File: kicad/gates/nquadstate/nquadstate.kicad_sch (KiCad schematic)
At the start: 11 parts, among them J1 Conn_01x03, J2 Conn_01x03, Q1 BSS8402DW-7-F, Q2 BSS8402DW-7-F, Q3 BSS8402DW-7-F

Commit message: update to kicad 9
Parts:
- J1, J2: Spice_Model Conn_01x03 -> (none); Spice_Netlist_Enabled N -> (none); Spice_Primitive J -> (none)
- Q1, Q2, Q3: Spice_Lib_File /lab/dev/tritium/library/TritiumSpice.lib -> (none); Spice_Model BSS8402DW -> (none); Spice_Netlist_Enabled Y -> (none); Spice_Primitive X -> (none)
- V1: value VDC -> 0; Spice_Model dc(0) -> (none); Spice_Netlist_Enabled Y -> (none); Spice_Primitive V -> (none)
- V2, V4: value VDC -> -5; Spice_Model dc(-5) -> (none); Spice_Netlist_Enabled Y -> (none); Spice_Primitive V -> (none)
- V3: value VDC -> 5; Spice_Model dc(5) -> (none); Spice_Netlist_Enabled Y -> (none); Spice_Primitive V -> (none)
