File: kicad/gates/sum/nconsensus.kicad_sch (KiCad schematic)
At the start: 4 parts, among them Q10 BSS8402DW-7-F, Q9 BSS8402DW-7-F

Commit message: update to kicad 9
Parts:
- Q10, Q9: Spice_Lib_File /lab/dev/tritium/library/TritiumSpice.lib -> (none); Spice_Model BSS8402DW -> (none); Spice_Netlist_Enabled Y -> (none); Spice_Primitive X -> (none)
