File: kicad/logic/analog_max/max.kicad_sch (KiCad schematic)
At the start: 8 parts, among them Q1 BSS8402DW-7-F, Q2 BSS8402DW-7-F

Commit message: update to kicad 9
Parts:
- A1, A2: Spice_Lib_File ${TRITIUM_LIB}/TritiumSpice.lib -> (none); Spice_Model Inverter -> (none); Spice_Netlist_Enabled Y -> (none); Spice_Primitive X -> (none)
- Q1, Q2: Spice_Lib_File ${TRITIUM_LIB}/TritiumSpice.lib -> (none); Spice_Model BSS8402DW -> (none); Spice_Primitive X -> (none)
- V1: value VDC -> 5; Spice_Model -5 -> (none); Spice_Netlist_Enabled Y -> (none); Spice_Primitive V -> (none)
- V2: value VDC -> -5; Spice_Model 0 -> (none); Spice_Netlist_Enabled Y -> (none); Spice_Primitive V -> (none)
- V3: value VDC -> 5; Spice_Model 5 -> (none); Spice_Netlist_Enabled Y -> (none); Spice_Primitive V -> (none)
- V4: value VDC -> -5; Spice_Model -5 -> (none); Spice_Netlist_Enabled Y -> (none); Spice_Primitive V -> (none)
