File: kicad/logic/sum/sum.kicad_sch (KiCad schematic)
At the start: 11 parts

Commit message: update to kicad 9
Parts:
- A1, A4, A6: Spice_Lib_File ${TRITIUM_LIB}/TritiumSpice.lib -> (none); Spice_Model NAny -> (none); Spice_Netlist_Enabled Y -> (none); Spice_Primitive X -> (none)
- A2: Spice_Lib_File ${TRITIUM_LIB}/TritiumSpice.lib -> (none); Spice_Model NConsensus -> (none); Spice_Netlist_Enabled Y -> (none); Spice_Primitive X -> (none)
- A3, A5, A7: Spice_Lib_File ${TRITIUM_LIB}/TritiumSpice.lib -> (none); Spice_Model Inverter -> (none); Spice_Netlist_Enabled Y -> (none); Spice_Primitive X -> (none)
- V1: value VDC -> 5; Spice_Model 5 -> (none); Spice_Netlist_Enabled Y -> (none); Spice_Primitive V -> (none)
- V2: value VDC -> 5; Spice_Model -5 -> (none); Spice_Netlist_Enabled Y -> (none); Spice_Primitive V -> (none)
- V3: value VDC -> 5; Spice_Model dc(5) -> (none); Spice_Netlist_Enabled Y -> (none); Spice_Primitive V -> (none)
- V4: value VDC -> -5; Spice_Model dc(-5) -> (none); Spice_Netlist_Enabled Y -> (none); Spice_Primitive V -> (none)
